Commit message: Update for KON414 Final Project

File: warthog_description/urdf/accessories.urdf.xacro (robot description, xacro)
@@ -52,3 +52,19 @@
     </xacro:if>
   </xacro:if>
+  <!-- 3D LiDAR Sensor -->
+  <xacro:include filename="accessories/lidar_3d.urdf.xacro" />
+  <xacro:if value="$(optenv WARTHOG_LIDAR_3D 1)">
+    <xacro:lidar_3d prefix="lidar_3d" parent_link="top_chassis_link">
+      <origin xyz="$(optenv WARTHOG_LIDAR_3D_OFFSET 0.0 0.0 0.1)"
+              rpy="$(optenv WARTHOG_LIDAR_3D_RPY 0 0 0)" />
+    </xacro:lidar_3d>
+  </xacro:if>
+  <!-- RGBD Camera -->
+  <xacro:include filename="accessories/rgbd_camera.urdf.xacro" />
+  <xacro:if value="$(optenv WARTHOG_RGBD_CAMERA 1)">
+    <xacro:rgbd_camera prefix="rgbd_camera" parent_link="top_chassis_link">
+      <origin xyz="$(optenv WARTHOG_RGBD_CAMERA_OFFSET 0.3 0.0 0.05)"
+              rpy="$(optenv WARTHOG_RGBD_CAMERA_RPY 0 0 0)" />
+    </xacro:rgbd_camera>
+  </xacro:if>
 </robot>

Commit message: Add lidar error

File: warthog_description/urdf/accessories.urdf.xacro (robot description, xacro)
@@ -56,6 +56,8 @@
   <xacro:if value="$(optenv WARTHOG_LIDAR_3D 1)">
     <xacro:lidar_3d prefix="lidar_3d" parent_link="top_chassis_link">
-      <origin xyz="$(optenv WARTHOG_LIDAR_3D_OFFSET 0.0 0.0 0.1)"
-              rpy="$(optenv WARTHOG_LIDAR_3D_RPY 0 0 0)" />
+      <!-- Intentional ±5% error in pose for sensor calibration testing -->
+      <!-- Original: xyz="0.0 0.0 0.1" rpy="0 0 0" -->
+      <origin xyz="$(optenv WARTHOG_LIDAR_3D_OFFSET 0.0 0.005 0.105)"
+              rpy="$(optenv WARTHOG_LIDAR_3D_RPY 0.0262 -0.0175 0.0349)" />
     </xacro:lidar_3d>
   </xacro:if>

Commit message: Update lidar and rgbd camera configuration.

File: warthog_description/urdf/accessories.urdf.xacro (robot description, xacro)
@@ -55,9 +55,9 @@
   <xacro:include filename="accessories/lidar_3d.urdf.xacro" />
   <xacro:if value="$(optenv WARTHOG_LIDAR_3D 1)">
-    <xacro:lidar_3d prefix="lidar_3d" parent_link="top_chassis_link">
-      <!-- Intentional ±5% error in pose for sensor calibration testing -->
-      <!-- Original: xyz="0.0 0.0 0.1" rpy="0 0 0" -->
-      <origin xyz="$(optenv WARTHOG_LIDAR_3D_OFFSET 0.0 0.005 0.105)"
-              rpy="$(optenv WARTHOG_LIDAR_3D_RPY 0.0262 -0.0175 0.0349)" />
+    <xacro:lidar_3d prefix="lidar_3d" parent_link="left_diff_unit_link">
+      <!-- Attached to left diff unit where antenna was located -->
+      <!-- Antenna position: xyz="-0.096 0.431 0.6635" (from warthog.urdf.xacro line 284) -->
+      <origin xyz="$(optenv WARTHOG_LIDAR_3D_OFFSET -0.2 0 0.540)"
+              rpy="$(optenv WARTHOG_LIDAR_3D_RPY 0 0 0)" />
     </xacro:lidar_3d>
   </xacro:if>
@@ -65,6 +65,9 @@
   <xacro:include filename="accessories/rgbd_camera.urdf.xacro" />
   <xacro:if value="$(optenv WARTHOG_RGBD_CAMERA 1)">
-    <xacro:rgbd_camera prefix="rgbd_camera" parent_link="top_chassis_link">
-      <origin xyz="$(optenv WARTHOG_RGBD_CAMERA_OFFSET 0.3 0.0 0.05)"
+    <xacro:rgbd_camera prefix="rgbd_camera" parent_link="left_diff_unit_link">
+      <!-- Attached to left diff unit where buttons were located -->
+      <!-- Buttons position: xyz="0.0395 0.4315 0.520" (from warthog.urdf.xacro line 255) -->
+      <!-- Rotate camera -90 degrees around z-axis to face forward -->
+      <origin xyz="$(optenv WARTHOG_RGBD_CAMERA_OFFSET 0.3 0 0.530)"
               rpy="0 0 0" />
     </xacro:rgbd_camera>

File: warthog_description/urdf/accessories/lidar_3d.urdf.xacro (robot description, xacro)
@@ -38,4 +38,5 @@
         <topic>${prefix}/points</topic>
         <update_rate>10</update_rate>
+        <gz_frame_id>${prefix}_link</gz_frame_id>
         <ray>
           <scan>

File: warthog_description/urdf/accessories/rgbd_camera.urdf.xacro (robot description, xacro)
@@ -44,4 +44,5 @@
     <gazebo reference="${prefix}_link">
       <sensor name="${prefix}_sensor" type="rgbd_camera">
+        <gz_frame_id>${prefix}_optical_frame</gz_frame_id>
         <camera>
           <horizontal_fov>2.0944</horizontal_fov>
